Commit message: bug with two robot states

File: install/kuka_urdf/share/kuka_urdf/urdf/kr210l150_romulus.urdf (robot description, URDF)
Before this commit: robot kuka_kr210, 8 links, 7 joints
Joints:
- removed joint joint_a1
- removed joint joint_a2
- removed joint joint_a3
- removed joint joint_a4
- removed joint joint_a5
- removed joint joint_a6
- removed joint link_6-tool0
- added joint romulus_joint_a1: type revolute, parent base_link, child link_1, origin xyz=-0.00262 0.00097586 0.33099 rpy=0 0 0, axis 0 0 1, limit lower=-3.228859205 upper=3.228859205 effort=0 velocity=2.146755039
- added joint romulus_joint_a2: type revolute, parent link_1, child link_2, origin xyz=0.35277 -0.037476 0.4192 rpy=0 0 0, axis 0 1 0, limit lower=-0.785398185 upper=1.483529905 effort=0 velocity=2.007128695
- added joint romulus_joint_a3: type revolute, parent link_2, child link_3, origin xyz=-9.8483E-05 -0.1475 1.2499 rpy=0 0 0, axis 0 1 0, limit lower=-3.66519153 upper=1.134464045 effort=0 velocity=1.954768816
- added joint romulus_joint_a4: type revolute, parent link_3, child link_4, origin xyz=0.95795 0.184 -0.055059 rpy=0 0 0, axis 1 0 0, limit lower=-6.10865255 upper=6.10865255 effort=0 velocity=3.124139447
- added joint romulus_joint_a5: type revolute, parent link_4, child link_5, origin xyz=0.542 0 0 rpy=0 0 0, axis 0 1 0, limit lower=-2.181661625 upper=2.181661625 effort=0 velocity=3.001966396
- added joint romulus_joint_a6: type revolute, parent link_5, child link_6, origin xyz=0.1925 0 0 rpy=0 0 0, axis 1 0 0, limit lower=-6.10865255 upper=6.10865255 effort=0 velocity=3.822271167
- added joint romulus_link_6-tool0: type fixed, parent link_6, child tool0, origin xyz=0.0375 0 -0.00023924 rpy=0 0 0

File: src/kuka_urdf/urdf/kr210l150_romulus.urdf (robot description, URDF)
Before this commit: robot kuka_kr210, 8 links, 7 joints
Joints:
- removed joint joint_a1
- removed joint joint_a2
- removed joint joint_a3
- removed joint joint_a4
- removed joint joint_a5
- removed joint joint_a6
- removed joint link_6-tool0
- added joint romulus_joint_a1: type revolute, parent base_link, child link_1, origin xyz=-0.00262 0.00097586 0.33099 rpy=0 0 0, axis 0 0 1, limit lower=-3.228859205 upper=3.228859205 effort=0 velocity=2.146755039
- added joint romulus_joint_a2: type revolute, parent link_1, child link_2, origin xyz=0.35277 -0.037476 0.4192 rpy=0 0 0, axis 0 1 0, limit lower=-0.785398185 upper=1.483529905 effort=0 velocity=2.007128695
- added joint romulus_joint_a3: type revolute, parent link_2, child link_3, origin xyz=-9.8483E-05 -0.1475 1.2499 rpy=0 0 0, axis 0 1 0, limit lower=-3.66519153 upper=1.134464045 effort=0 velocity=1.954768816
- added joint romulus_joint_a4: type revolute, parent link_3, child link_4, origin xyz=0.95795 0.184 -0.055059 rpy=0 0 0, axis 1 0 0, limit lower=-6.10865255 upper=6.10865255 effort=0 velocity=3.124139447
- added joint romulus_joint_a5: type revolute, parent link_4, child link_5, origin xyz=0.542 0 0 rpy=0 0 0, axis 0 1 0, limit lower=-2.181661625 upper=2.181661625 effort=0 velocity=3.001966396
- added joint romulus_joint_a6: type revolute, parent link_5, child link_6, origin xyz=0.1925 0 0 rpy=0 0 0, axis 1 0 0, limit lower=-6.10865255 upper=6.10865255 effort=0 velocity=3.822271167
- added joint romulus_link_6-tool0: type fixed, parent link_6, child tool0, origin xyz=0.0375 0 -0.00023924 rpy=0 0 0
