Commit message: two working robots

File: install/kuka_urdf/share/kuka_urdf/urdf/kr210l150_remus.urdf (robot description, URDF)
Before this commit: robot remus, 8 links, 7 joints
Links:
- removed link remus_base_link
- removed link remus_link_1
- removed link remus_link_2
- removed link remus_link_3
- removed link remus_link_4
- removed link remus_link_5
- removed link remus_link_6
- removed link remus_tool0
- added link a_base_link; collision mesh filename=package://kuka_urdf/meshes/collision/base_link.stl; visual mesh filename=package://kuka_urdf/meshes/visual/base_link.dae
- added link a_link_1, mass 1385.5; collision mesh filename=package://kuka_urdf/meshes/collision/link_1.stl; visual mesh filename=package://kuka_urdf/meshes/visual/link_1.dae
- added link a_link_2, mass 958.62; collision mesh filename=package://kuka_urdf/meshes/collision/link_2.stl; visual mesh filename=package://kuka_urdf/meshes/visual/link_2.dae
- added link a_link_3, mass 710.03; collision mesh filename=package://kuka_urdf/meshes/collision/link_3.stl; visual mesh filename=package://kuka_urdf/meshes/visual/link_3.dae
- added link a_link_4, mass 173.73; collision mesh filename=package://kuka_urdf/meshes/collision/link_4.stl; visual mesh filename=package://kuka_urdf/meshes/visual/link_4.dae
- added link a_link_5, mass 72.17; collision mesh filename=package://kuka_urdf/meshes/collision/link_5.stl; visual mesh filename=package://kuka_urdf/meshes/visual/link_5.dae
- added link a_link_6, mass 6.3154; collision mesh filename=package://kuka_urdf/meshes/collision/link_6.stl; visual mesh filename=package://kuka_urdf/meshes/visual/link_6.dae
- added link a_tool0; visual cylinder length=0.1 radius=0.005; visual cylinder length=0.1 radius=0.005
Joints:
- removed joint remus_joint_a1
- removed joint remus_joint_a2
- removed joint remus_joint_a3
- removed joint remus_joint_a4
- removed joint remus_joint_a5
- removed joint remus_joint_a6
- removed joint remus_link_6-tool0
- added joint a_joint_a1: type revolute, parent a_base_link, child a_link_1, origin xyz=-0.00262 0.00097586 0.33099 rpy=0 0 0, axis 0 0 1, limit lower=-3.228859205 upper=3.228859205 effort=0 velocity=2.146755039
- added joint a_joint_a2: type revolute, parent a_link_1, child a_link_2, origin xyz=0.35277 -0.037476 0.4192 rpy=0 0 0, axis 0 1 0, limit lower=-0.785398185 upper=1.483529905 effort=0 velocity=2.007128695
- added joint a_joint_a3: type revolute, parent a_link_2, child a_link_3, origin xyz=-9.8483E-05 -0.1475 1.2499 rpy=0 0 0, axis 0 1 0, limit lower=-3.66519153 upper=1.134464045 effort=0 velocity=1.954768816
- added joint a_joint_a4: type revolute, parent a_link_3, child a_link_4, origin xyz=0.95795 0.184 -0.055059 rpy=0 0 0, axis 1 0 0, limit lower=-6.10865255 upper=6.10865255 effort=0 velocity=3.124139447
- added joint a_joint_a5: type revolute, parent a_link_4, child a_link_5, origin xyz=0.542 0 0 rpy=0 0 0, axis 0 1 0, limit lower=-2.181661625 upper=2.181661625 effort=0 velocity=3.001966396
- added joint a_joint_a6: type revolute, parent a_link_5, child a_link_6, origin xyz=0.1925 0 0 rpy=0 0 0, axis 1 0 0, limit lower=-6.10865255 upper=6.10865255 effort=0 velocity=3.822271167
- added joint a_link_6-tool0: type fixed, parent a_link_6, child a_tool0, origin xyz=0.0375 0 -0.00023924 rpy=0 0 0

Commit message: working two robot display

File: install/kuka_urdf/share/kuka_urdf/urdf/kr210l150_remus.urdf (robot description, URDF)
Before this commit: robot remus, 8 links, 7 joints
Links:
- removed link base_link
- removed link link_1
- removed link link_2
- removed link link_3
- removed link link_4
- removed link link_5
- removed link link_6
- removed link tool0
- added link a_base_link; collision mesh filename=package://kuka_urdf/meshes/collision/base_link.stl; visual mesh filename=package://kuka_urdf/meshes/visual/base_link.dae
- added link a_link_1, mass 1385.5; collision mesh filename=package://kuka_urdf/meshes/collision/link_1.stl; visual mesh filename=package://kuka_urdf/meshes/visual/link_1.dae
- added link a_link_2, mass 958.62; collision mesh filename=package://kuka_urdf/meshes/collision/link_2.stl; visual mesh filename=package://kuka_urdf/meshes/visual/link_2.dae
- added link a_link_3, mass 710.03; collision mesh filename=package://kuka_urdf/meshes/collision/link_3.stl; visual mesh filename=package://kuka_urdf/meshes/visual/link_3.dae
- added link a_link_4, mass 173.73; collision mesh filename=package://kuka_urdf/meshes/collision/link_4.stl; visual mesh filename=package://kuka_urdf/meshes/visual/link_4.dae
- added link a_link_5, mass 72.17; collision mesh filename=package://kuka_urdf/meshes/collision/link_5.stl; visual mesh filename=package://kuka_urdf/meshes/visual/link_5.dae
- added link a_link_6, mass 6.3154; collision mesh filename=package://kuka_urdf/meshes/collision/link_6.stl; visual mesh filename=package://kuka_urdf/meshes/visual/link_6.dae
- added link a_tool0; visual cylinder length=0.1 radius=0.005; visual cylinder length=0.1 radius=0.005
Joints:
- removed joint joint_a1
- removed joint joint_a2
- removed joint joint_a3
- removed joint joint_a4
- removed joint joint_a5
- removed joint joint_a6
- removed joint link_6-tool0
- added joint a_joint_a1: type revolute, parent a_base_link, child a_link_1, origin xyz=-0.00262 0.00097586 0.33099 rpy=0 0 0, axis 0 0 1, limit lower=-3.228859205 upper=3.228859205 effort=0 velocity=2.146755039
- added joint a_joint_a2: type revolute, parent a_link_1, child a_link_2, origin xyz=0.35277 -0.037476 0.4192 rpy=0 0 0, axis 0 1 0, limit lower=-0.785398185 upper=1.483529905 effort=0 velocity=2.007128695
- added joint a_joint_a3: type revolute, parent a_link_2, child a_link_3, origin xyz=-9.8483E-05 -0.1475 1.2499 rpy=0 0 0, axis 0 1 0, limit lower=-3.66519153 upper=1.134464045 effort=0 velocity=1.954768816
- added joint a_joint_a4: type revolute, parent a_link_3, child a_link_4, origin xyz=0.95795 0.184 -0.055059 rpy=0 0 0, axis 1 0 0, limit lower=-6.10865255 upper=6.10865255 effort=0 velocity=3.124139447
- added joint a_joint_a5: type revolute, parent a_link_4, child a_link_5, origin xyz=0.542 0 0 rpy=0 0 0, axis 0 1 0, limit lower=-2.181661625 upper=2.181661625 effort=0 velocity=3.001966396
- added joint a_joint_a6: type revolute, parent a_link_5, child a_link_6, origin xyz=0.1925 0 0 rpy=0 0 0, axis 1 0 0, limit lower=-6.10865255 upper=6.10865255 effort=0 velocity=3.822271167
- added joint a_link_6-tool0: type fixed, parent a_link_6, child a_tool0, origin xyz=0.0375 0 -0.00023924 rpy=0 0 0

Commit message: corrected urdf files but not working movement

File: install/kuka_urdf/share/kuka_urdf/urdf/kr210l150_remus.urdf (robot description, URDF)
Before this commit: robot remus, 8 links, 7 joints
Links:
- removed link a_base_link
- removed link a_link_1
- removed link a_link_2
- removed link a_link_3
- removed link a_link_4
- removed link a_link_5
- removed link a_link_6
- removed link a_tool0
- added link remus_base_link; collision mesh filename=package://kuka_urdf/meshes/collision/base_link.stl; visual mesh filename=package://kuka_urdf/meshes/visual/base_link.dae
- added link remus_link_1, mass 1385.5; collision mesh filename=package://kuka_urdf/meshes/collision/link_1.stl; visual mesh filename=package://kuka_urdf/meshes/visual/link_1.dae
- added link remus_link_2, mass 958.62; collision mesh filename=package://kuka_urdf/meshes/collision/link_2.stl; visual mesh filename=package://kuka_urdf/meshes/visual/link_2.dae
- added link remus_link_3, mass 710.03; collision mesh filename=package://kuka_urdf/meshes/collision/link_3.stl; visual mesh filename=package://kuka_urdf/meshes/visual/link_3.dae
- added link remus_link_4, mass 173.73; collision mesh filename=package://kuka_urdf/meshes/collision/link_4.stl; visual mesh filename=package://kuka_urdf/meshes/visual/link_4.dae
- added link remus_link_5, mass 72.17; collision mesh filename=package://kuka_urdf/meshes/collision/link_5.stl; visual mesh filename=package://kuka_urdf/meshes/visual/link_5.dae
- added link remus_link_6, mass 6.3154; collision mesh filename=package://kuka_urdf/meshes/collision/link_6.stl; visual mesh filename=package://kuka_urdf/meshes/visual/link_6.dae
- added link remus_tool0; visual cylinder length=0.1 radius=0.005; visual cylinder length=0.1 radius=0.005
Joints:
- removed joint a_joint_a1
- removed joint a_joint_a2
- removed joint a_joint_a3
- removed joint a_joint_a4
- removed joint a_joint_a5
- removed joint a_joint_a6
- removed joint a_link_6-tool0
- added joint remus_joint_a1: type revolute, parent remus_base_link, child remus_link_1, origin xyz=-0.00262 0.00097586 0.33099 rpy=0 0 0, axis 0 0 1, limit lower=-3.228859205 upper=3.228859205 effort=0 velocity=2.146755039
- added joint remus_joint_a2: type revolute, parent remus_link_1, child remus_link_2, origin xyz=0.35277 -0.037476 0.4192 rpy=0 0 0, axis 0 1 0, limit lower=-0.785398185 upper=1.483529905 effort=0 velocity=2.007128695
- added joint remus_joint_a3: type revolute, parent remus_link_2, child remus_link_3, origin xyz=-9.8483E-05 -0.1475 1.2499 rpy=0 0 0, axis 0 1 0, limit lower=-3.66519153 upper=1.134464045 effort=0 velocity=1.954768816
- added joint remus_joint_a4: type revolute, parent remus_link_3, child remus_link_4, origin xyz=0.95795 0.184 -0.055059 rpy=0 0 0, axis 1 0 0, limit lower=-6.10865255 upper=6.10865255 effort=0 velocity=3.124139447
- added joint remus_joint_a5: type revolute, parent remus_link_4, child remus_link_5, origin xyz=0.542 0 0 rpy=0 0 0, axis 0 1 0, limit lower=-2.181661625 upper=2.181661625 effort=0 velocity=3.001966396
- added joint remus_joint_a6: type revolute, parent remus_link_5, child remus_link_6, origin xyz=0.1925 0 0 rpy=0 0 0, axis 1 0 0, limit lower=-6.10865255 upper=6.10865255 effort=0 velocity=3.822271167
- added joint remus_link_6-tool0: type fixed, parent remus_link_6, child remus_tool0, origin xyz=0.0375 0 -0.00023924 rpy=0 0 0

File: install/kuka_urdf/share/kuka_urdf/urdf/kr210l150_romulus.urdf (robot description, URDF)
Before this commit: robot romulus, 8 links, 7 joints
Links:
- removed link base_link
- removed link link_1
- removed link link_2
- removed link link_3
- removed link link_4
- removed link link_5
- removed link link_6
- removed link tool0
- added link romulus_base_link; collision mesh filename=package://kuka_urdf/meshes/collision/base_link.stl; visual mesh filename=package://kuka_urdf/meshes/visual/base_link.dae
- added link romulus_link_1, mass 1385.5; collision mesh filename=package://kuka_urdf/meshes/collision/link_1.stl; visual mesh filename=package://kuka_urdf/meshes/visual/link_1.dae
- added link romulus_link_2, mass 958.62; collision mesh filename=package://kuka_urdf/meshes/collision/link_2.stl; visual mesh filename=package://kuka_urdf/meshes/visual/link_2.dae
- added link romulus_link_3, mass 710.03; collision mesh filename=package://kuka_urdf/meshes/collision/link_3.stl; visual mesh filename=package://kuka_urdf/meshes/visual/link_3.dae
- added link romulus_link_4, mass 173.73; collision mesh filename=package://kuka_urdf/meshes/collision/link_4.stl; visual mesh filename=package://kuka_urdf/meshes/visual/link_4.dae
- added link romulus_link_5, mass 72.17; collision mesh filename=package://kuka_urdf/meshes/collision/link_5.stl; visual mesh filename=package://kuka_urdf/meshes/visual/link_5.dae
- added link romulus_link_6, mass 6.3154; collision mesh filename=package://kuka_urdf/meshes/collision/link_6.stl; visual mesh filename=package://kuka_urdf/meshes/visual/link_6.dae
- added link romulus_tool0; visual cylinder length=0.1 radius=0.005; visual cylinder length=0.1 radius=0.005
Joints:
- joint romulus_joint_a1: child link_1 -> romulus_link_1; parent base_link -> romulus_base_link
- joint romulus_joint_a2: child link_2 -> romulus_link_2; parent link_1 -> romulus_link_1
- joint romulus_joint_a3: child link_3 -> romulus_link_3; parent link_2 -> romulus_link_2
- joint romulus_joint_a4: child link_4 -> romulus_link_4; parent link_3 -> romulus_link_3
- joint romulus_joint_a5: child link_5 -> romulus_link_5; parent link_4 -> romulus_link_4
- joint romulus_joint_a6: child link_6 -> romulus_link_6; parent link_5 -> romulus_link_5
- joint romulus_link_6-tool0: child tool0 -> romulus_tool0; parent link_6 -> romulus_link_6
